Commit message: DartIntegration version 2

File: src/Magnum/DartIntegration/Test/urdf/test_multi_mesh.urdf (robot description, URDF)
Before this commit: robot texture_urdf, 2 links, 1 joints
Links:
- removed link world
- link base_link: geometry collision mesh filename=suzanne.blend; visual mesh filename=suzanne.blend
Joints:
- removed joint arm_to_world_fixed
